File: EMK/EMK.kicad_pcb (KiCad board)
At the start: 2 copper layers, 117 parts, among them Q1 Si2371EDS, Q2 Si2371EDS, SW1 SW_Nidec_CAS-120A1, SW10 MX3, SW11 MX7, SW12 MX11, SW13 MX15, SW14 MX4, SW15 MX8, SW16 MX12, SW17 MX16, SW18 SW_Push, SW19 SW_Nidec_CAS-120A1, SW2 MX1, SW3 MX5, SW4 MX9, SW5 MX13, SW6 MX2, SW7 MX6, SW8 MX10, SW9 MX14, U1 nRF52840-QFAA, U2 15nH, U3 TPS62822DLC, U4 USBLC6-2SC6, U5 TP4057, Y1 Crystal_32.768kHz, Y2 Crystal_32mHz

Commit message: Roteamento da MCU e posicionamento
Parts:
- added AE1: Antenna, RF_Antenna:Johanson_2450AT43F0100, B.Cu at (42.6, 71.0)
- C1, C10, C11, C12, C13, C14, C15, C16, C17, C18, C19, C2, C20, C21, C3, C4, C5, C6, C7, C8, C9, D1, D2, D3, L1, L2, L3, Q1, Q2, R1, R10, R11, R13, R2, R3, R4, R5, R6, R7, R8, R9, SW1, SW19, U1, U2, U3, U4, U5, Y2: moved to B.Cu
- D10, D11, D12, D13, D14, D15, D16, D17, D18, D19, D4, D5, D6, D7, D8, D9: footprint Diode_SMD:D_0201_0603Metric -> Diode_SMD:D_0603_1608Metric
- SW14: footprint Button_Switch_Keyboard:SW_Cherry_MX_1.25u_Plate -> Button_Switch_Keyboard:SW_Cherry_MX_6.25u_PCB
- SW3, SW4: footprint Button_Switch_Keyboard:SW_Cherry_MX_1.25u_Plate -> Button_Switch_Keyboard:SW_Cherry_MX_2.00u_Vertical_Plate
- Y1: footprint Crystal:Crystal_AT310_D3.0mm_L10.0mm_Horizontal -> Crystal:Crystal_SMD_2012-2Pin_2.0x1.2mm; moved to B.Cu
- moved SW3 215.3 mm to (147.5, 117.4)
- moved SW2 214.6 mm to (117.5, 124.9)
- moved SW14 213.3 mm to (105.0, 149.9)
- moved SW6 195.7 mm to (92.5, 124.9)
- moved D5 192.9 mm to (152.5, 112.5), turned to -90 degrees
- moved SW10 183.7 mm to (67.5, 124.9)
- moved D16 182.5 mm to (112.5, 147.5), turned to 90 degrees
- moved SW4 179.0 mm to (147.5, 77.4)
- moved D4 178.3 mm to (125.0, 122.5), turned to -90 degrees
- moved SW7 177.1 mm to (117.5, 105.0)
- moved D6 173.2 mm to (152.5, 72.5), turned to -90 degrees
- moved D9 162.7 mm to (125.3, 102.5), turned to -90 degrees
- moved D7 161.5 mm to (150.0, 42.5), turned to -90 degrees
- moved D8 158.7 mm to (100.0, 122.5), turned to -90 degrees
- moved SW11 157.5 mm to (92.5, 104.9)
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Connections:
- net ANT_TRACE renamed Net-(AE1-A)
Routing:
- net ANT_BT: track 0.00 -> 31.5 mm
- net Net-(AE1-A): track 0.00 -> 20.7 mm
- net VSS_PA: track 0.00 -> 12.4 mm
- net Net-(U1-DCC): track 0.00 -> 10.8 mm
- net Net-(U1-P0.04/AIN2): track 0.00 -> 9.02 mm
- net Net-(U1-DEC3): track 0.00 -> 7.93 mm
- net Net-(U1-XC2): track 0.00 -> 7.26 mm
- net Net-(U1-XC1): track 0.00 -> 7.26 mm
- net Net-(U1-DEC1): track 0.00 -> 6.98 mm
- net Net-(U1-P0.00/XL1): track 0.00 -> 6.53 mm
- net Net-(U1-P0.01/XL2): track 0.00 -> 6.40 mm
- net Net-(L1-Pad1): track 0.00 -> 6.40 mm
- net Net-(C20-Pad1): track 0.00 -> 6.20 mm
- net Net-(C10-Pad1): track 0.00 -> 5.63 mm
- net Net-(U1-DEC4): track 0.00 -> 4.11 mm
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Other:
- board outline added: 130 x 150 mm

Commit message: feat: realiza o roteamento das trilhas da matriz e dos leds.
Signed-off-by: Paulo Santos <prms@ic.ufal.br>
Parts:
- added J1: USB_C_Receptacle_USB2.0_14P, Connector_USB:USB_C_Receptacle_XKB_U262-16XN-4BVC11, B.Cu at (129.9, 28.7)
- added J2: Conn_01x02_Socket, Connector_PinHeader_2.54mm:PinHeader_1x02_P2.54mm_Horizontal, B.Cu at (119.4, 32.6)
- C22, C23, C24, C25, C26, C27, C28, C29, C30, C31, C32, C33, C34, C35, C36, C37, D10, D11, D12, D13, D14, D15, D16, D17, D18, D19, D4, D5, D6, D7, D8, D9: moved to B.Cu
- D2, D3, R6: moved to F.Cu
- D20, D21, D22, D23, D24, D25, D26, D27, D28, D29, D30, D31, D32, D33, D34, D35: value WS2812B -> SK6812MINI; footprint LED_SMD:LED_WS2812B_PLCC4_5.0x5.0mm_P3.2mm -> LED:SK6812MINI-E-PLCC4_3.2x2.8mm; moved to B.Cu
- L1, U2: footprint Inductor_SMD:L_7.3x7.3_H4.5 -> Inductor_SMD:L_0603_1608Metric
- SW10, SW2, SW6: footprint Button_Switch_Keyboard:SW_Cherry_MX_1.25u_Plate -> Button_Switch_Keyboard:SW_Cherry_MX_1.25u_PCB
- SW11, SW12, SW13, SW15, SW16, SW17, SW5, SW9: footprint Button_Switch_Keyboard:SW_Cherry_MX_1.25u_Plate -> Button_Switch_Keyboard:SW_Cherry_MX_1.00u_Plate
- SW14: footprint Button_Switch_Keyboard:SW_Cherry_MX_6.25u_PCB -> Button_Switch_Keyboard:SW_Cherry_MX_1.25u_PCB
- SW18: footprint Button_Switch_SMD:SW_SPST_B3S-1000 -> Button_Switch_SMD:SW_SPST_B3U-1000P; moved to B.Cu
- SW3, SW4: footprint Button_Switch_Keyboard:SW_Cherry_MX_2.00u_Vertical_Plate -> Button_Switch_Keyboard:SW_Cherry_MX_1.50u_PCB
- SW7, SW8: footprint Button_Switch_Keyboard:SW_Cherry_MX_1.25u_Plate -> Button_Switch_Keyboard:SW_Cherry_MX_1.50u_PCB
- U5: footprint Package_TO_SOT_SMD:TSOT-23-5 -> Package_TO_SOT_SMD:TSOT-23-6
- moved D29 182.3 mm to (54.1, 106.2), turned to 180 degrees
- moved C34 174.3 mm to (60.5, 103.6), turned to -90 degrees
- moved D28 172.8 mm to (51.8, 87.4), turned to 180 degrees
- moved D33 167.5 mm to (101.8, 106.5), turned to 180 degrees
- moved C35 166.1 mm to (84.3, 103.6), turned to -90 degrees
- moved C36 161.2 mm to (108.0, 103.6), turned to -90 degrees
- moved D31 160.2 mm to (78.0, 106.5), turned to 180 degrees
- moved C37 159.6 mm to (131.9, 103.6), turned to -90 degrees
- moved D32 157.8 mm to (94.6, 87.3), turned to 180 degrees
- moved D24 152.4 mm to (52.0, 68.5), turned to 180 degrees
- moved D30 152.0 mm to (70.8, 87.5), turned to 180 degrees
- moved C30 151.1 mm to (57.9, 84.6), turned to -90 degrees
- moved D35 149.3 mm to (125.4, 106.5), turned to 180 degrees
- moved C31 143.0 mm to (77.0, 84.4), turned to -90 degrees
- moved D34 137.3 mm to (123.2, 87.3), turned to 180 degrees
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Connections:
- C1 pad 1: Net-(C1-Pad1) -> VSS_PA
- C10 pad 1: Net-(C10-Pad1) -> VDD_NRF
- C10 pad 2: Net-(C10-Pad2) -> VSS_PA
- C11 pad 2: Net-(C10-Pad2) -> VSS_PA
- C12 pad 1: Net-(C12-Pad1) -> VSS_PA
- C13 pad 2: Net-(C13-Pad2) -> VSS_PA
- C14 pad 2: GND -> VSS_PA
- C15 pad 2: GND -> VSS_PA
- C17 pad 2: GND -> VSS_PA
- C18 pad 2: GND -> VSS_PA
- C19 pad 2: GND -> VSS_PA
- C2 pad 1: Net-(C1-Pad1) -> VSS_PA
- C20 pad 2: GND -> VSS_PA
- C22 pad 1: GND -> VSS_PA
- C23 pad 1: GND -> VSS_PA
- C24 pad 1: GND -> VSS_PA
- C25 pad 1: GND -> VSS_PA
- C26 pad 1: GND -> VSS_PA
- C27 pad 1: GND -> VSS_PA
- C28 pad 1: GND -> VSS_PA
- C29 pad 1: GND -> VSS_PA
- C3 pad 1: Net-(C3-Pad1) -> VSS_PA
- C30 pad 1: GND -> VSS_PA
- C31 pad 1: GND -> VSS_PA
- C32 pad 1: GND -> VSS_PA
- C33 pad 1: GND -> VSS_PA
- C34 pad 1: GND -> VSS_PA
- C35 pad 1: GND -> VSS_PA
- C36 pad 1: GND -> VSS_PA
- C37 pad 1: GND -> VSS_PA
- C4 pad 1: Net-(C3-Pad1) -> VSS_PA
- C6 pad 2: Net-(C6-Pad2) -> VSS_PA
- C8 pad 1: Net-(C12-Pad1) -> VSS_PA
- C9 pad 1: Net-(C9-Pad1) -> VDD_NRF
- C9 pad 2: Net-(C10-Pad2) -> VSS_PA
- D20 pad 3: GND -> VSS_PA
- D21 pad 3: GND -> VSS_PA
- D22 pad 3: GND -> VSS_PA
- D23 pad 3: GND -> VSS_PA
- D24 pad 3: GND -> VSS_PA
- D25 pad 3: GND -> VSS_PA
- D26 pad 3: GND -> VSS_PA
- D27 pad 3: GND -> VSS_PA
- D28 pad 3: GND -> VSS_PA
- D29 pad 3: GND -> VSS_PA
- D29 pad 4: Net-(D28-DOUT) -> Net-(D29-DIN)
- D30 pad 3: GND -> VSS_PA
- D30 pad 4: Net-(D29-DOUT) -> Net-(D28-DOUT)
- D31 pad 3: GND -> VSS_PA
- D31 pad 4: Net-(D30-DOUT) -> Net-(D29-DOUT)
- D32 pad 3: GND -> VSS_PA
- D32 pad 4: Net-(D31-DOUT) -> Net-(D30-DOUT)
- D33 pad 3: GND -> VSS_PA
- D33 pad 4: Net-(D32-DOUT) -> Net-(D31-DOUT)
- D34 pad 2: Net-(D34-DOUT) -> Net-(D29-DIN)
- D34 pad 3: GND -> VSS_PA
- D34 pad 4: Net-(D33-DOUT) -> Net-(D32-DOUT)
- D35 pad 3: GND -> VSS_PA
- D35 pad 4: Net-(D34-DOUT) -> Net-(D33-DOUT)
- D36 pad 1: GND -> VSS_PA
- R1 pad 2: GND -> VSS_PA
- R11 pad 1: GND -> VSS_PA
- R2 pad 2: GND -> VSS_PA
- R3 pad 2: GND -> VSS_PA
- R5 pad 2: GND -> VSS_PA
- R7 pad 2: GND -> VSS_PA
- R8 pad 2: GND -> VSS_PA
- SW18 pad 2: GND -> VSS_PA
- U1 pad 17: Net-(C9-Pad1) -> VDD_NRF
- U1 pad 25: Net-(C10-Pad1) -> VDD_NRF
- U3 pad 3: GND -> VSS_PA
- U3 pad 5: GND -> VSS_PA
- U5 pad 2: GND -> VSS_PA
Routing:
- net RGB_VDD: track 0.00 -> 438.8 mm, vias 0 -> 17
- net COL3: track 0.00 -> 204.1 mm, vias 0 -> 3
- net COL2: track 0.00 -> 189.2 mm, vias 0 -> 3
- net COL0: track 0.00 -> 169.1 mm, vias 0 -> 1
- net COL1: track 0.00 -> 166.5 mm, vias 0 -> 3
- net ROW0: track 0.00 -> 133.9 mm, vias 0 -> 2
- net RGB_SIG: track 0.00 -> 113.0 mm, vias 0 -> 2
- net ROW1: track 0.00 -> 109.6 mm, vias 0 -> 2
- net ROW3: track 0.00 -> 103.2 mm, vias 0 -> 2
- net ROW2: track 0.00 -> 103.0 mm
- net Net-(D27-DOUT): track 0.00 -> 93.8 mm, vias 0 -> 2
- net Net-(D29-DIN): track 0.00 -> 90.9 mm, vias 0 -> 2
- net Net-(D23-DOUT): track 0.00 -> 87.6 mm, vias 0 -> 4
- net VDD_NRF: track 3.27 -> 64.6 mm, vias 0 -> 6
- net NRST: track 0.00 -> 39.6 mm, vias 0 -> 2
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- added copper zone on In2.Cu, net VSS_PA
Other:
- board size 130 x 150 mm -> 112.2 x 87.7 mm
- copper layers 2 -> 4

Commit message: Roteamento
Parts:
- moved C6 4.86 mm to (141.9, 73.7)
- moved U2 0.78 mm to (132.6, 59.6)
- moved R11 0.62 mm to (145.8, 55.2)
- moved C13 0.45 mm to (133.9, 56.9)
- moved C12 0.11 mm to (138.2, 66.1), turned to 0 degrees
Connections:
- C1 pad 1: VSS_PA -> GND
- C10 pad 2: VSS_PA -> GND
- C11 pad 2: VSS_PA -> GND
- C12 pad 1: VSS_PA -> GND
- C13 pad 2: VSS_PA -> GND
- C14 pad 2: VSS_PA -> GND
- C15 pad 2: VSS_PA -> GND
- C17 pad 2: VSS_PA -> GND
- C18 pad 2: VSS_PA -> GND
- C19 pad 2: VSS_PA -> GND
- C2 pad 1: VSS_PA -> GND
- C20 pad 2: VSS_PA -> GND
- C21 pad 2: VSS_PA -> GND
- C22 pad 1: VSS_PA -> GND
- C23 pad 1: VSS_PA -> GND
- C24 pad 1: VSS_PA -> GND
- C25 pad 1: VSS_PA -> GND
- C26 pad 1: VSS_PA -> GND
- C27 pad 1: VSS_PA -> GND
- C28 pad 1: VSS_PA -> GND
- C29 pad 1: VSS_PA -> GND
- C3 pad 1: VSS_PA -> GND
- C30 pad 1: VSS_PA -> GND
- C31 pad 1: VSS_PA -> GND
- C32 pad 1: VSS_PA -> GND
- C33 pad 1: VSS_PA -> GND
- C34 pad 1: VSS_PA -> GND
- C35 pad 1: VSS_PA -> GND
- C36 pad 1: VSS_PA -> GND
- C37 pad 1: VSS_PA -> GND
- C4 pad 1: VSS_PA -> GND
- C5 pad 1: Net-(C5-Pad1) -> GND
- C6 pad 2: VSS_PA -> GND
- C7 pad 2: Net-(C7-Pad2) -> GND
- C8 pad 1: VSS_PA -> GND
- C9 pad 2: VSS_PA -> GND
- D20 pad 3: VSS_PA -> GND
- D21 pad 3: VSS_PA -> GND
- D22 pad 3: VSS_PA -> GND
- D23 pad 3: VSS_PA -> GND
- D24 pad 3: VSS_PA -> GND
- D25 pad 3: VSS_PA -> GND
- D26 pad 3: VSS_PA -> GND
- D27 pad 3: VSS_PA -> GND
- D28 pad 3: VSS_PA -> GND
- D29 pad 3: VSS_PA -> GND
- D30 pad 3: VSS_PA -> GND
- D31 pad 3: VSS_PA -> GND
- D32 pad 3: VSS_PA -> GND
- D33 pad 3: VSS_PA -> GND
- D34 pad 3: VSS_PA -> GND
- D35 pad 3: VSS_PA -> GND
- D36 pad 1: VSS_PA -> GND
- J1 pad A1: VSS_PA -> GND
- J1 pad A12: VSS_PA -> GND
- J1 pad B1: VSS_PA -> GND
- J1 pad B12: VSS_PA -> GND
- J1 pad S1: VSS_PA -> GND
- J2 pad 1: VSS_PA -> GND
- R1 pad 2: VSS_PA -> GND
- R11 pad 1: VSS_PA -> GND
- R2 pad 2: VSS_PA -> GND
- R3 pad 2: VSS_PA -> GND
- R5 pad 2: VSS_PA -> GND
- R7 pad 2: VSS_PA -> GND
- R8 pad 2: VSS_PA -> GND
- SW18 pad 2: VSS_PA -> GND
- U1 pad 32: VSS_PA -> GND
- U1 pad 45: VSS_PA -> GND
- U1 pad 49: VSS_PA -> GND
- U3 pad 3: VSS_PA -> GND
- U3 pad 5: VSS_PA -> GND
- U5 pad 2: VSS_PA -> GND
Routing:
- net GND: track 0.00 -> 100.9 mm, vias 0 -> 58
- net MCU_VDD_RGB: track 0.00 -> 33.9 mm, vias 0 -> 2
- net ANT_BT: track 0.00 -> 29.5 mm
- net COL0: track 169.1 -> 150.6 mm
- net RGB_VDD: track 438.8 -> 456.8 mm
- net VSS_PA: track 8.93 -> 0.00 mm, vias 3 -> 0
- net Net-(C20-Pad1): track 0.00 -> 6.85 mm
- net Net-(AE1-A): track 0.00 -> 5.17 mm
- net Net-(U1-DEC3): track 1.88 -> 6.40 mm
- net Net-(J1-CC1): track 0.00 -> 4.49 mm
- net Net-(J1-CC2): track 0.00 -> 3.44 mm
- net Net-(L1-Pad1): track 0.00 -> 2.36 mm
- net Net-(C13-Pad1): track 0.00 -> 2.13 mm
- net ROW3: track 103.2 -> 105.3 mm
- net RGB_SIG: track 113.0 -> 114.6 mm
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- added copper zone on In1.Cu, net GND
- removed copper zone on In2.Cu, net VSS_PA

Commit message: Ajusta a PCI
Adiciona as trilhas faltantes.
Parts:
- added J3: Conn_ARM_JTAG_SWD_10, LED:ARM_SWD_SMD_TH, B.Cu at (110.0, 28.4)
- added SW20: Mode Switch, LED:MODE-SWITCH-SLW12745474ARAD, F.Cu at (98.3, 29.0)
- moved R13 46.6 mm to (91.6, 31.8), turned to 0 degrees
- moved C11 13.5 mm to (146.7, 57.7), turned to 90 degrees
- moved C10 7.38 mm to (145.0, 75.5), turned to -90 degrees
- moved R11 0.60 mm to (145.8, 54.6)
Routing:
- net MATRIX_M1: track 0.00 -> 82.8 mm, vias 0 -> 1
- net VDD_NRF: track 65.4 -> 140.4 mm, vias 6 -> 9
- net MATRIX_M2: track 0.00 -> 74.3 mm, vias 0 -> 1
- net MATRIX_M3: track 0.00 -> 73.4 mm, vias 0 -> 1
- net SWDIO: track 0.00 -> 62.7 mm, vias 0 -> 2
- net SWCLK: track 0.00 -> 61.8 mm, vias 0 -> 2
- net VBUS: track 34.2 -> 91.1 mm
- net NRST: track 39.6 -> 78.8 mm
- net VBAT: track 31.9 -> 66.6 mm, vias 2 -> 4
- net Net-(D3-K): track 0.00 -> 31.0 mm, vias 0 -> 1
- net Net-(D2-K): track 0.00 -> 26.6 mm, vias 0 -> 3
- net GND: track 100.9 -> 110.6 mm, vias 58 -> 60
- net COL0: track 150.6 -> 140.9 mm
- net Net-(Q1-D): track 0.00 -> 9.03 mm, vias 0 -> 2
- net Net-(R13-Pad2): track 0.00 -> 2.83 mm
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