File: EMK/untitled.kicad_sch (KiCad schematic)
At the start: 0 parts

Commit message: feat: organiza o esquemático e adiciona as labels aos blocos.
Signed-off-by: Paulo Santos <prms@ic.ufal.br>
Parts:
- added D10, D11, D12, D13, D14, D15, D16, D17, D18, D19, D4, D5, D6, D7, D8, D9: D, symbol Device:D
- added SW10: MX3, symbol Switch:SW_Push
- added SW11: MX7, symbol Switch:SW_Push
- added SW12: MX11, symbol Switch:SW_Push
- added SW13: MX15, symbol Switch:SW_Push
- added SW14: MX4, symbol Switch:SW_Push
- added SW15: MX8, symbol Switch:SW_Push
- added SW16: MX12, symbol Switch:SW_Push
- added SW17: MX16, symbol Switch:SW_Push
- added SW2: MX1, symbol Switch:SW_Push
- added SW3: MX5, symbol Switch:SW_Push
- added SW4: MX9, symbol Switch:SW_Push
- added SW5: MX13, symbol Switch:SW_Push
- added SW6: MX2, symbol Switch:SW_Push
- added SW7: MX6, symbol Switch:SW_Push
- added SW8: MX10, symbol Switch:SW_Push
- added SW9: MX14, symbol Switch:SW_Push
Connections:
- new net: D18.2 (A), SW16.1
- new net: D5.2 (A), SW3.1
- new net: D17.2 (A), SW15.1
- new net: D19.2 (A), SW17.1
- new net: D6.2 (A), SW4.1
- new net: D11.2 (A), SW9.1
- new net: D10.2 (A), SW8.1
- new net: D9.2 (A), SW7.1
- new net: D16.2 (A), SW14.1
- new net: D15.2 (A), SW13.1
- new net: D4.2 (A), SW2.1
- new net: D8.2 (A), SW6.1
- new net: D14.2 (A), SW12.1
- new net: D13.2 (A), SW11.1
- new net: D12.2 (A), SW10.1
- new net: D7.2 (A), SW5.1
- new net COL0: SW2.2, SW3.2, SW4.2, SW5.2
- new net COL1: SW6.2, SW7.2, SW8.2, SW9.2
- new net COL2: SW10.2, SW11.2, SW12.2, SW13.2
- new net COL3: SW14.2, SW15.2, SW16.2, SW17.2
- new net ROW0: D12.1 (K), D16.1 (K), D4.1 (K), D8.1 (K)
- new net ROW1: D13.1 (K), D17.1 (K), D5.1 (K), D9.1 (K)
- new net ROW2: D10.1 (K), D14.1 (K), D18.1 (K), D6.1 (K)
- new net ROW3: D11.1 (K), D15.1 (K), D19.1 (K), D7.1 (K)
Other:
- title: (none) -> EMK
