File: EMK/_autosave-EMK.kicad_pcb (KiCad board)
At the start: 4 copper layers, 112.2 x 87.7 mm, 122 parts, among them J1 USB_C_Receptacle_USB2.0_14P, J2 Conn_01x02_Socket, J3 Conn_ARM_JTAG_SWD_10, Q1 Si2371EDS, Q2 Si2371EDS, SW1 SW_Nidec_CAS-120A1, SW10 MX3, SW11 MX7, SW12 MX11, SW13 MX15, SW14 MX4, SW15 MX8, SW16 MX12, SW17 MX16, SW18 SW_Push, SW19 SW_Nidec_CAS-120A1, SW2 MX1, SW20 Mode Switch, SW3 MX5, SW4 MX9, SW5 MX13, SW6 MX2, SW7 MX6, SW8 MX10, SW9 MX14, U1 nRF52840-QFAA, U2 15nH, U3 TPS62822DLC, U4 USBLC6-2SC6, U5 TP4057, Y1 Crystal_32.768kHz, Y2 Crystal_32mHz

Commit message: Alimentação
Parts:
- moved J2 11.4 mm to (121.3, 43.8)
Routing:
- net VBAT: track 68.1 -> 28.9 mm
- net MCU_VDD_RGB: track 34.4 -> 25.0 mm
- net VDD_NRF: track 140.4 -> 139.0 mm
- net Net-(U3-FB): track 12.6 -> 12.1 mm
- added copper zone on In2.Cu, net RGB_VDD
- added copper zone on In2.Cu, net VBAT
