File: EMK/EMK.kicad_sch (KiCad schematic)
At the start: 52 parts, among them J1 USB_C_Receptacle_USB2.0_14P, J2 Conn_01x02_Socket, J3 Conn_ARM_JTAG_SWD_10, Q1 Si2371EDS, Q2 Si2371EDS, SW1 SW_Nidec_CAS-120A1, SW18 SW_Push, SW19 SW_Nidec_CAS-120A1, U1 nRF52840-QFAA, U2 15nH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

Commit message: Remap tracement
Parts:
- C20: footprint Capacitor_SMD:C_0603_1608Metric -> Capacitor_SMD:C_0402_1005Metric
- L3: footprint Inductor_SMD:L_0603_1608Metric -> Inductor_SMD:L_0402_1005Metric
- L4: footprint Inductor_SMD:L_0603_1608Metric -> Inductor_SMD:L_0402_1005Metric_Pad0.77x0.64mm_HandSolder
Connections:
- net MATRIX_M1: now also U1.9 (P1.09/TRACEDATA3); no longer U1.15 (P0.17)
- net MATRIX_M2: now also U1.10 (P0.11/TRACEDATA2); no longer U1.14 (P0.14)
- net MATRIX_M3: now also U1.11 (P0.12/TRACEDATA1); no longer U1.13 (P0.13)
- net RGB_ON: now also U1.8 (P1.08); no longer U1.7 (P0.08)
- net RGB_SIG: now also U1.7 (P0.08); no longer U1.8 (P1.08)
- net ROW2: no longer U1.20 (P0.21)
Changed lines of the file:
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@@
 	(wire
 		(pts
+			(xy 74.93 133.35) (xy 76.2 133.35)
+		)
+		(stroke
+			(width 0)
+			(type default)
+		)
+	)
+	(wire
+		(pts
 			(xy 146.05 41.91) (xy 146.05 35.56)
 		)
@@
 	(wire
 		(pts
-			(xy 85.09 43.18) (xy 85.09 62.23)
-		)
-		(stroke
-			(width 0)
-			(type default)
-		)
-	)
-	(wire
-		(pts
 			(xy 355.6 109.22) (xy 344.17 109.22)
 		)
@@
 	(wire
 		(pts
-			(xy 336.55 109.22) (xy 336.55 118.11)
+			(xy 74.93 118.11) (xy 74.93 133.35)
 		)
 		(stroke
@@
 	(wire
 		(pts
-			(xy 39.37 90.17) (xy 36.83 90.17)
+			(xy 69.85 139.7) (xy 69.85 118.11)
 		)
 		(stroke
@@
 	(wire
 		(pts
-			(xy 251.46 114.3) (xy 251.46 127)
+			(xy 336.55 109.22) (xy 336.55 118.11)
 		)
 		(stroke
@@
 	(wire
 		(pts
-			(xy 54.61 121.92) (xy 54.61 118.11)
+			(xy 39.37 90.17) (xy 36.83 90.17)
+		)
+		(stroke
+			(width 0)
+			(type default)
+		)
+	)
+	(wire
+		(pts
+			(xy 251.46 114.3) (xy 251.46 127)
 		)
 		(stroke
@@
 	(wire
 		(pts
-			(xy 87.63 53.34) (xy 87.63 62.23)
+			(xy 54.61 121.92) (xy 54.61 118.11)
 		)
 		(stroke
@@
 	(wire
 		(pts
-			(xy 80.01 49.53) (xy 80.01 62.23)
-		)
-		(stroke
-			(width 0)
-			(type default)
-		)
-	)
-	(wire
-		(pts
 			(xy 151.13 120.65) (xy 151.13 123.19)
 		)
@@
 	(wire
 		(pts
-			(xy 52.07 49.53) (xy 52.07 62.23)
-		)
-		(stroke
-			(width 0)
-			(type default)
-		)
-	)
-	(wire
-		(pts
 			(xy 243.84 132.08) (xy 243.84 127)
 		)
@@
 	(wire
 		(pts
+			(xy 72.39 127) (xy 72.39 118.11)
+		)
+		(stroke
+			(width 0)
+			(type default)
+		)
+	)
+	(wire
+		(pts
 			(xy 40.64 121.92) (xy 41.91 121.92)
 		)
@@
 		)
 	)
-	(global_label "MATRIX_M2"
-		(shape input)
-		(at 82.55 62.23 90)
-		(fields_autoplaced yes)
-		(effects
-			(font
-				(size 1.27 1.27)
-			)
-			(justify left)
-		)
-		(property "Intersheetrefs" "${INTERSHEET_REFS}"
-			(at 82.55 49.0244 90)
-			(effects
-				(font
-					(size 1.27 1.27)
-				)
-				(justify left)
-				(hide yes)
-			)
-		)
-	)
 	(global_label "VBAT"
 		(shape input)
@@
 	(global_label "RGB_SIG"
 		(shape input)
-		(at 52.07 49.53 90)
+		(at 87.63 62.23 90)
 		(fields_autoplaced yes)
 		(effects
@@
 		)
 		(property "Intersheetrefs" "${INTERSHEET_REFS}"
-			(at 52.07 38.6829 90)
+			(at 87.63 51.3829 90)
 			(effects
 				(font
@@
 	(global_label "MATRIX_M1"
 		(shape input)
-		(at 80.01 49.53 90)
+		(at 69.85 139.7 270)
 		(fields_autoplaced yes)
 		(effects
@@
 				(size 1.27 1.27)
 			)
-			(justify left)
+			(justify right)
 		)
 		(property "Intersheetrefs" "${INTERSHEET_REFS}"
-			(at 80.01 36.3244 90)
+			(at 69.85 152.9056 90)
 			(effects
 				(font
 					(size 1.27 1.27)
 				)
-				(justify left)
+				(justify right)
 				(hide yes)
 			)
@@
 		)
 	)
-	(global_label "MATRIX_M3"
-		(shape input)
-		(at 85.09 43.18 90)
-		(fields_autoplaced yes)
-		(effects
-			(font
-				(size 1.27 1.27)
-			)
-			(justify left)
-		)
-		(property "Intersheetrefs" "${INTERSHEET_REFS}"
-			(at 85.09 29.9744 90)
-			(effects
-				(font
-					(size 1.27 1.27)
-				)
-				(justify left)
-				(hide yes)
-			)
-		)
-	)
 	(global_label "RGB_ON"
 		(shape input)
@@
 		)
 	)
-	(global_label "ROW2"
+	(global_label "MATRIX_M2"
 		(shape input)
-		(at 72.39 62.23 90)
+		(at 72.39 127 270)
 		(fields_autoplaced yes)
 		(effects
@@
 				(size 1.27 1.27)
 			)
-			(justify left)
+			(justify right)
 		)
 		(property "Intersheetrefs" "${INTERSHEET_REFS}"
-			(at 72.39 53.9834 90)
+			(at 72.39 140.2056 90)
 			(effects
 				(font
 					(size 1.27 1.27)
 				)
-				(justify left)
+				(justify right)
 				(hide yes)
 			)
@@
 		)
 	)
+	(global_label "MATRIX_M3"
+		(shape input)
+		(at 76.2 133.35 270)
+		(fields_autoplaced yes)
+		(effects
+			(font
+				(size 1.27 1.27)
+			)
+			(justify right)
+		)
+		(property "Intersheetrefs" "${INTERSHEET_REFS}"
+			(at 76.2 146.5556 90)
+			(effects
+				(font
+					(size 1.27 1.27)
+				)
+				(justify right)
+				(hide yes)
+			)
+		)
+	)
 	(global_label "VBUS"
 		(shape input)
@@
 	(global_label "RGB_ON"
 		(shape input)
-		(at 87.63 53.34 90)
+		(at 52.07 62.23 90)
 		(fields_autoplaced yes)
 		(effects
@@
 		)
 		(property "Intersheetrefs" "${INTERSHEET_REFS}"
-			(at 87.63 42.9162 90)
+			(at 52.07 51.8062 90)
 			(effects
 				(font
@@
 			)
 		)
-		(property "Footprint" "Inductor_SMD:L_0603_1608Metric"
+		(property "Footprint" "Inductor_SMD:L_0402_1005Metric"
 			(at 237.49 200.66 0)
 			(effects
@@
 			)
 		)
-		(property "Footprint" "Capacitor_SMD:C_0603_1608Metric"
+		(property "Footprint" "Capacitor_SMD:C_0402_1005Metric"
 			(at 262.89 199.6948 0)
 			(effects
@@
 			)
 		)
-		(property "Footprint" "Inductor_SMD:L_0603_1608Metric"
+		(property "Footprint" "Inductor_SMD:L_0402_1005Metric_Pad0.77x0.64mm_HandSolder"
 			(at 245.11 204.47 0)
 			(effects
