File: EMK/EMK.kicad_sch (KiCad schematic)
At the start: 52 parts, among them J1 USB_C_Receptacle_USB2.0_14P, J2 Conn_01x02_Socket, J3 Conn_ARM_JTAG_SWD_10, Q1 Si2371EDS, Q2 Si2371EDS, SW1 SW_Nidec_CAS-120A1, SW18 SW_Push, SW19 SW_Nidec_CAS-120A1, U1 nRF52840-QFAA, U2 15nH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

Commit message: Refatora a antena
Ajusta a antena.
Parts:
- C20: value 1pF -> 1.2pF
- L3: value 3.9nH -> 3.3nH
Changed lines of the file:
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@@
 			)
 		)
-		(property "Value" "3.9nH"
+		(property "Value" "3.3nH"
 			(at 237.49 198.12 90)
 			(effects
@@
 			)
 		)
-		(property "Value" "1pF"
+		(property "Value" "1.2pF"
 			(at 259.08 195.58 90)
 			(effects
